Commit message: Added gazebo_imu_sensor

File: diffbot_description/urdf/diffbot.urdf.xacro (robot description, xacro)
@@ -36,4 +36,19 @@
                       base_props="${base_props}" >
   </xacro:wheel>
+  <gazebo reference="imu_link">
+    <sensor type="imu" name="my_imu">
+    <always_on>true</always_on>
+    <!-- Publish at 30 hz -->
+    <update_rate>30</update_rate>
+    <plugin name="my_imu_plugin" filename="libgazebo_ros_imu_sensor.so">
+      <ros>
+        <!-- Will publish to /imu/data -->
+        <namespace>/imu</namespace>
+        <argument>~/out:=data</argument>
+      </ros>
+      <!-- frame_name ommited, will be "my_link" -->
+    </plugin>
+    </sensor>
+  </gazebo>
   <!-- Motors -->
   <xacro:motor prefix="right" reflect="-1"

File: diffbot_description/urdf/include/common_sensors.xacro (robot description, xacro)
@@ -175,72 +175,3 @@
   </gazebo>
 </xacro:macro>
-<xacro:macro name="imu_sensor" params=" *joint_origin parent_link sensor_prop">
-  <xacro:property name="mesh"
-     value="${sensor_prop['imu']['mesh']}"/>
-  <link name="imu_link">
-    <xacro:if value="${mesh != '' }" >
-      <visual>
-        <origin xyz="0 0 0" rpy="0 0 0"/>
-        <geometry>
-          <mesh filename="package://${package_name}/meshes/sensors/${mesh}" scale="${sensor_prop['imu']['scale']}" />
-        </geometry>
-        <material name="dark_grey"/>
-      </visual>
-    </xacro:if>
-    <xacro:if value="${mesh == '' }" >
-      <visual>
-        <origin xyz="0 0 0" rpy="0 0 0"/>
-        <geometry>
-          <cylinder radius="${sensor_prop['imu']['radius']}" length="${sensor_prop['imu']['length']}"/>
-        </geometry>
-        <material name="red"/>
-      </visual>
-    </xacro:if>
-    <collision>
-      <origin xyz="0 0 0" rpy="0 0 0"/>
-      <geometry>
-        <box size="0.01 0.01 0.01"/>
-      </geometry>
-    </collision>
-    <xacro:box_inertia m="${sensor_prop['imu']['mass']}"
-                       x="${sensor_prop['imu']['size']['x']}"
-                       y="${sensor_prop['imu']['size']['y']}"
-                       z="${sensor_prop['imu']['size']['y']}" />
-    <!-- Todo delete visual>
-      <origin xyz="0 0 0" rpy="0 0 0"/>
-      <geometry>
-        <box size="0.01 0.01 0.01"/>
-      </geometry>
-    </visual>
-    <inertial>
-      <mass value="1e-5" />
-      <origin xyz="0 0 0" rpy="0 0 0"/>
-      <inertia ixx="1e-6" ixy="0" ixz="0" iyy="1e-6" iyz="0" izz="1e-6" />
-    </inertial-->
-  </link>
-  <gazebo reference="imu_link">
-    <material>Gazebo/Yellow</material>
-  </gazebo>
-  <joint name="imu_joint" type="fixed">
-    <axis xyz="0 1 0" />
-    <xacro:insert_block name="joint_origin" />
-    <parent link="${parent_link}"/>
-    <child link="imu_link"/>
-  </joint>
-  <gazebo reference="imu_link">
-    <sensor type="imu" name="my_imu">
-    <always_on>true</always_on>
-    <!-- Publish at 30 hz -->
-    <update_rate>30</update_rate>
-    <plugin name="my_imu_plugin" filename="libgazebo_ros_imu_sensor.so">
-      <ros>
-        <!-- Will publish to /imu/data -->
-        <namespace>/imu</namespace>
-        <argument>~/out:=data</argument>
-      </ros>
-      <!-- frame_name ommited, will be "my_link" -->
-    </plugin>
-    </sensor>
-  </gazebo>
-</xacro:macro>
 </robot>

File: diffbot_description/urdf/include/robot.gazebo.xacro (robot description, xacro)
@@ -11,4 +11,16 @@
     </gazebo>
   </xacro:macro>
+  <!-- imu_sensor plugin-->
+  <gazebo>
+    <plugin name="imu_plugin" filename="libgazebo_ros_imu.so">
+      <alwaysOn>true</alwaysOn>
+      <bodyName>base_link</bodyName>
+      <topicName>imu</topicName>
+      <serviceName>imu_service</serviceName>
+      <gaussianNoise>0.0</gaussianNoise>
+      <updateRate>20.0</updateRate>
+    </plugin>
+  </gazebo>
+  <!-- sonar_sensor plugin-->
   <!-- xacro to set the friction for the wheel. This patch was taken from the MIR
   repository.

Commit message: Added simulated IMU (cleaned code) and simulated ultrasonic sensor (with model 3d integrated).

File: diffbot_description/urdf/diffbot.urdf.xacro (robot description, xacro)
@@ -50,4 +50,21 @@
                    enable_gpu="${sensor_prop['laser']['enable_gpu']}">
   </xacro:laser>
+  <xacro:imu_sensor parent_link="base_link" sensor_prop="${sensor_prop}">
+                   <origin xyz="0 0 0" rpy="0 0 0"/>
+  </xacro:imu_sensor>
+    <!--Added Ultrasonic sensor frame -->
+  <link name="ultrasonic_link">
+    <visual>
+      <origin rpy="0.0 0 ${-pi/2}" xyz="0 0 0"/>
+      <geometry>
+        <mesh filename="package://diffbot_description/meshes/sensors/ultrasonic.dae"/>
+      </geometry>
+    </visual>
+  </link>
+   <joint name="base_to_ultrasonic" type="fixed">
+    <parent link="base_link"/>
+    <child link="ultrasonic_link"/>
+    <origin xyz="0.065 0 0.01"/>
+  </joint>
   <!-- Gazebo -->
   <xacro:gazebo_ros_control robotNamespace="/diffbot">

File: diffbot_description/urdf/include/common_sensors.xacro (robot description, xacro)
@@ -175,3 +175,104 @@
   </gazebo>
 </xacro:macro>
+<xacro:macro name="imu_sensor" params="parent_link sensor_prop *joint_origin">
+  <xacro:property name="mesh"
+     value="${sensor_prop['imu']['mesh']}"/>
+  <link name="imu_link">
+    <xacro:if value="${mesh != '' }" >
+      <visual>
+        <origin xyz="0 0 0" rpy="0 0 0"/>
+        <geometry>
+          <mesh filename="package://${package_name}/meshes/sensors/${mesh}" scale="${sensor_prop['imu']['scale']}" />
+        </geometry>
+        <material name="dark_grey"/>
+      </visual>
+    </xacro:if>
+    <xacro:if value="${mesh == '' }" >
+      <visual>
+        <origin xyz="0 0 0" rpy="0 0 0"/>
+        <geometry>
+          <cylinder radius="${sensor_prop['imu']['radius']}" length="${sensor_prop['imu']['length']}"/>
+        </geometry>
+        <material name="red"/>
+      </visual>
+    </xacro:if>
+    <collision>
+      <origin xyz="0 0 0" rpy="0 0 0"/>
+      <geometry>
+        <box size="0.01 0.01 0.01"/>
+      </geometry>
+    </collision>
+    <xacro:box_inertia m="${sensor_prop['imu']['mass']}"
+                       x="${sensor_prop['imu']['size']['x']}"
+                       y="${sensor_prop['imu']['size']['y']}"
+                       z="0" />
+  </link>
+  <gazebo reference="imu_link">
+    <material>Gazebo/Yellow</material>
+  </gazebo>
+  <joint name="imu_joint" type="fixed">
+    <axis xyz="0 1 0" />
+    <xacro:insert_block name="joint_origin" />
+    <parent link="${parent_link}"/>
+    <child link="imu_link"/>
+  </joint>
+  <gazebo reference="imu_link">
+    <gravity>true</gravity>
+    <sensor name="imu_sensor" type="imu">
+      <always_on>true</always_on>
+      <update_rate>100</update_rate>
+      <visualize>true</visualize>
+      <topic>alpha_bot/imu</topic>
+      <plugin filename="libgazebo_ros_imu_sensor.so" name="imu_plugin">
+        <topicName>sensor/imu</topicName>
+        <bodyName>imu_link</bodyName>
+        <updateRateHZ>30.0</updateRateHZ>
+        <gaussianNoise>0.005</gaussianNoise>
+        <xyzOffset>0 0 0</xyzOffset>
+        <rpyOffset>0 0 0</rpyOffset>
+        <frameName>imu_link</frameName>
+        <initialOrientationAsReference>false</initialOrientationAsReference>
+      </plugin>
+      <pose>0 0 0 0 0 0</pose>
+    </sensor>
+  </gazebo>
+  <!--Added ultrasonic sensor-->
+ <gazebo reference="ultrasonic_link">
+   <sensor type="ray" name="TeraRanger">
+      <pose>0 0 0 0 0 0</pose>
+      <visualize>true</visualize>
+      <update_rate>50</update_rate>
+      <ray>
+         <scan>
+            <horizontal>
+               <samples>10</samples>
+               <resolution>1</resolution>
+               <min_angle>-0.14835</min_angle>
+               <max_angle>0.14835</max_angle>
+            </horizontal>
+            <vertical>
+               <samples>10</samples>
+               <resolution>1</resolution>
+               <min_angle>-0.14835</min_angle>
+               <max_angle>0.14835</max_angle>
+            </vertical>
+         </scan>
+         <range>
+            <min>0.01</min>
+            <max>2</max>
+            <resolution>0.02</resolution>
+         </range>
+      </ray>
+      <plugin filename="libgazebo_ros_range.so" name="gazebo_ros_range">
+         <gaussianNoise>0.005</gaussianNoise>
+         <alwaysOn>true</alwaysOn>
+         <updateRate>50</updateRate>
+         <topicName>sensor/range</topicName>
+         <frameName>ultrasonic_link</frameName>
+         <radiation>INFRARED</radiation>
+         <fov>0.2967</fov>
+      </plugin>
+   </sensor>
+   </gazebo>
+</xacro:macro>
 </robot>

File: diffbot_description/urdf/include/robot.gazebo.xacro (robot description, xacro)
@@ -11,16 +11,15 @@
     </gazebo>
   </xacro:macro>
-  <!-- imu_sensor plugin-->
-  <gazebo>
-    <plugin name="imu_plugin" filename="libgazebo_ros_imu.so">
-      <alwaysOn>true</alwaysOn>
-      <bodyName>base_link</bodyName>
-      <topicName>imu</topicName>
-      <serviceName>imu_service</serviceName>
-      <gaussianNoise>0.0</gaussianNoise>
-      <updateRate>20.0</updateRate>
-    </plugin>
-  </gazebo>
-  <!-- sonar_sensor plugin-->
+  <!-- range_sensor plugin
+  <plugin name="gazebo_range_sensor" filename="libgazebo_ros_range.so" >
+        <alwaysOn>true</alwaysOn>
+        <updateRate>5</updateRate>
+        <bodyName>base_link</bodyName>
+        <topicName>range/fl</topicName>
+        <frameName>range_front_left_frame</frameName>
+        <fov>0.1</fov>
+        <radiation>ultrasound</radiation>
+        <gaussianNoise>0.005</gaussianNoise>
+   </plugin> -->
   <!-- xacro to set the friction for the wheel. This patch was taken from the MIR
   repository.
